File: EtherEar.sch (KiCad schematic (older format))
At the start: 21 parts

Commit message: labels
Parts:
- gave numbers to parts that had none: 7
Changed lines of the file:
@@
 $EndComp
 $Comp
-L Device:LED D?
+L Device:LED D1
 U 1 1 5E65D6C4
 P 6400 2700
-F 0 "D?" V 6439 2583 50  0000 R CNN
+F 0 "D1" V 6439 2583 50  0000 R CNN
 F 1 "LED" V 6348 2583 50  0000 R CNN
 F 2 "" H 6400 2700 50  0001 C CNN
@@
 	1    0    0    -1
 $EndComp
-$Comp
-L Device:LED D?
-U 1 1 5E6615A0
-P 6700 2700
-F 0 "D?" V 6739 2583 50  0000 R CNN
-F 1 "LED" V 6648 2583 50  0000 R CNN
-F 2 "" H 6700 2700 50  0001 C CNN
-F 3 "~" H 6700 2700 50  0001 C CNN
-	1    6700 2700
-	0    -1   -1   0
-$EndComp
 Wire Wire Line
 	6700 2050 6700 2150
@@
 $EndComp
 $Comp
-L Device:LED D?
+L Device:LED D3
 U 1 1 5E661CFD
 P 7000 2700
-F 0 "D?" V 7039 2583 50  0000 R CNN
+F 0 "D3" V 7039 2583 50  0000 R CNN
 F 1 "LED" V 6948 2583 50  0000 R CNN
 F 2 "" H 7000 2700 50  0001 C CNN
@@
 $EndComp
 $Comp
-L Device:LED D?
+L Device:LED D4
 U 1 1 5E6676D5
 P 7300 2700
-F 0 "D?" V 7339 2583 50  0000 R CNN
+F 0 "D4" V 7339 2583 50  0000 R CNN
 F 1 "LED" V 7248 2583 50  0000 R CNN
 F 2 "" H 7300 2700 50  0001 C CNN
@@
 $EndComp
 $Comp
-L Device:LED D?
+L Device:LED D5
 U 1 1 5E6676E9
 P 7600 2700
-F 0 "D?" V 7639 2583 50  0000 R CNN
+F 0 "D5" V 7639 2583 50  0000 R CNN
 F 1 "LED" V 7548 2583 50  0000 R CNN
 F 2 "" H 7600 2700 50  0001 C CNN
@@
 $EndComp
 $Comp
-L Device:LED D?
+L Device:LED D6
 U 1 1 5E6676FD
 P 7900 2700
-F 0 "D?" V 7939 2583 50  0000 R CNN
+F 0 "D6" V 7939 2583 50  0000 R CNN
 F 1 "LED" V 7848 2583 50  0000 R CNN
 F 2 "" H 7900 2700 50  0001 C CNN
@@
 $EndComp
 $Comp
-L Device:C C?
+L Device:C C1
 U 1 1 5E680E6D
 P 4950 2050
-F 0 "C?" H 5065 2096 50  0000 L CNN
+F 0 "C1" H 5065 2096 50  0000 L CNN
 F 1 "10u" H 5065 2005 50  0000 L CNN
 F 2 "" H 4988 1900 50  0001 C CNN
@@
 	-1   0    0    1
 $EndComp
+$Comp
+L Device:LED D2
+U 1 1 5E6615A0
+P 6700 2700
+F 0 "D2" V 6739 2583 50  0000 R CNN
+F 1 "LED" V 6648 2583 50  0000 R CNN
+F 2 "" H 6700 2700 50  0001 C CNN
+F 3 "~" H 6700 2700 50  0001 C CNN
+	1    6700 2700
+	0    -1   -1   0
+$EndComp
 $EndSCHEMATC
